File: Archivos Kicad/Motor_Board.kicad_pcb (KiCad board)
At the start: 2 copper layers, 66 parts, among them IC1 L298, P1 Motor A, P2 VDD Motor, P3 Motor B, SW1 Switch_SPDT_x2, U2 7805

Commit message: Segunda versión del pcb. Ubicación de componentes de acuerdo a las medidas de la plantilla de la Edu Ciaa.
Parts:
- added MP?: Plantilla_EDU-CIAA, Motor_Board:Plantilla_EDU-CIAA, F.Cu at (151.5, 91.0)
- added XA?: Plantilla_Poncho_Izquierda, Motor_Board:Plantilla_Poncho_Plantilla_Poncho_Izquierda, F.Cu at (330.0, 89.0)
- moved F1 264.4 mm to (382.2, 46.3)
- moved F2 264.4 mm to (382.2, 46.3)
- moved F3 264.4 mm to (382.2, 46.3)
- moved R16 122.6 mm to (92.6, 123.6), turned to 270 degrees
- moved P3 96.3 mm to (81.5, 81.0), turned to 90 degrees
- moved P1 92.0 mm to (81.5, 70.0), turned to 90 degrees
- moved R8 91.3 mm to (106.0, 61.5), turned to 270 degrees
- moved R14 90.2 mm to (121.5, 58.5), turned to 90 degrees
- moved R12 85.8 mm to (106.0, 77.0), turned to 270 degrees
- moved R13 85.0 mm to (111.0, 58.5), turned to 90 degrees
- moved R19 82.8 mm to (144.5, 58.5), turned to 90 degrees
- moved R11 82.1 mm to (106.0, 123.6), turned to 270 degrees
- moved R3 80.2 mm to (92.6, 46.5), turned to 270 degrees
- moved D1 80.1 mm to (101.0, 47.0), turned to 180 degrees
- moved D7 79.8 mm to (127.5, 118.5), turned to 90 degrees
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Routing:
- net /GPIO3: track 0.00 -> 66.9 mm, vias 0 -> 1
- net /GPIO5: track 0.00 -> 53.5 mm, vias 0 -> 1
- net /GPIO2: track 0.00 -> 42.5 mm
- net /GPIO7: track 0.00 -> 40.2 mm
- net /GPIO8: track 0.00 -> 14.6 mm
- net /IN1: track 0.00 -> 14.1 mm, vias 0 -> 1
- net Net-(D4-Pad1): track 0.00 -> 10.4 mm
- net VDD: track 0.00 -> 9.38 mm, vias 0 -> 4
- net Net-(D3-Pad1): track 0.00 -> 9.26 mm
- net Net-(D1-Pad1): track 0.00 -> 9.06 mm
- net Net-(D2-Pad1): track 0.00 -> 8.96 mm
- net Net-(D21-Pad1): track 0.00 -> 8.04 mm
- net /IN3: track 0.00 -> 7.93 mm, vias 0 -> 1
- net Net-(D15-Pad1): track 0.00 -> 7.24 mm
- net /IN2: track 0.00 -> 6.51 mm
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Other:
- board outline added: 94.5 x 109 mm
- net class Default: clearance 0.2 -> 0.254; trace_width 0.25 -> 0.254; via_dia 0.6 -> 1.016; via_drill 0.4 -> 0.508
- rule trace_clearance: 0.2 -> 0.254
- rule trace_min: 0.2 -> 0.254
- rule via_min_drill: 0.3 -> 0.508
- rule via_min_size: 0.4 -> 1.016

Commit message: Segunda versión del PCB.
Parts:
- added G***: LOGO, Motor_Board:Logo_Poncho, F.Cu at (140.1, 133.0)
- added G101: Logo_OSHWA, Motor_Board:Logo_OSHWA, F.Cu at (128.1, 133.9)
- moved MP? 116.4 mm to (267.8, 87.7)
- moved P1 74.8 mm to (145.0, 109.5)
- moved P3 65.6 mm to (145.0, 97.5)
- moved D5 33.8 mm to (148.9, 59.6), turned to 90 degrees
- moved D6 32.1 mm to (146.0, 59.5)
- moved D16 32.0 mm to (147.5, 46.0)
- moved R13 32.0 mm to (143.0, 59.5)
- moved P2 23.0 mm to (81.5, 82.0)
- moved SW1 19.5 mm to (81.5, 70.5), turned to 270 degrees
- moved D13 16.4 mm to (138.3, 59.5), turned to 90 degrees
- moved C5 16.3 mm to (113.0, 131.0)
- moved D14 16.2 mm to (135.6, 59.5), turned to 90 degrees
- moved D12 16.1 mm to (125.2, 59.5), turned to 90 degrees
- moved D10 14.7 mm to (114.7, 59.5), turned to 90 degrees
- moved D11 12.0 mm to (128.0, 59.5)
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Routing:
- net GNDA: track 0.00 -> 89.4 mm
- net /GPIO0: track 2.34 -> 82.5 mm, vias 1 -> 0
- net (no net): track 1.78 -> 11.5 mm, vias 1 -> 0
- net Net-(D16-Pad2): track 0.00 -> 4.21 mm
- net /ENB: track 1.64 -> 4.18 mm
- net /IN4: track 1.84 -> 0.00 mm, vias 1 -> 0
- net Net-(D4-Pad1): track 10.4 -> 9.10 mm
- net Net-(D15-Pad1): track 7.24 -> 8.24 mm
- net Net-(D1-Pad1): track 9.06 -> 8.35 mm
- net Net-(D3-Pad1): track 9.26 -> 8.58 mm
- net Net-(D2-Pad1): track 8.96 -> 8.38 mm
Other:
- board size 94.5 x 109 mm -> 76.9 x 105 mm
